File: pcb/coin20mm/coin20mm.kicad_pcb (KiCad board)
At the start: 2 copper layers, 27.9 x 23.6 mm, 11 parts, among them CN1 1X4-CLEANBIG

Commit message: readme for pcb
Parts:
- removed U$4: , coin20mm:ADAFRUIT_5MM
