File: pcb/pcb_lora/pcb_lora.kicad_pcb (KiCad board)
At the start: 2 copper layers, 25.4 x 29.2 mm, 18 parts, among them U1 RFM69HCW, U2 74HC4050D, U3 AP2112K-3.3, X1 uFL/SMA

Commit message: readme for pcb
Parts:
- removed U$8: , pcb_lora:ADAFRUIT_3.5MM
